File: Schemes/glove3.sch (EAGLE design)
At the start: 69 parts, among them IC1 ATMEGA32U4-MU, IC2 74HC595D, IC3 74HC595D, SW1 SPST_TACT-KMR2, T1 BC847, T2 BC847, T3 BC847, T4 BC847, T5 BC847, T6 BC847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

Commit message: 
Parts:
- removed IC2, IC3: 74HC595D, 74xx-eu:74HC595D
- removed JP1: (no value), microbuilder:HEADER-1X16ROUND
- removed JP3: (no value), microbuilder:HEADER-1X12
- removed R11, R12, R13, R14, R15, R16, R17, R18, R19, R20, R21, R22, R23: (no value), SparkFun-Resistors:RESISTOR1206
- removed T1, T2, T3, T4, T5, T6: BC847, transistor:BC847
- removed T10, T11, T12, T13, T7, T8, T9: (no value), transistor:BC857C-PNP-SOT23-BEC
- added IC4, IC5: PCF8574TS, micro-philips:PCF8574TS
- added J1, J2, J3: (no value), con-lsta:JU05
- added R24, R25, R26, R27, R28, R29, R30, R31, R32, R33, R34, R35, R36, R37, R38: (no value), SparkFun-Resistors:RESISTOR1206
- added SV1, SV2, SV3: (no value), con-lstb:MA05-1
- added T14, T15, T16, T17, T18, T19, T20, T28: (no value), transistor:BC857C-PNP-SOT23-BEC
- added T21, T22, T23, T24, T25, T26, T27: BC847, transistor:BC847
Connections:
- removed net 0: JP1.3
- removed net 1: JP1.2
- removed net 10: JP3.7
- removed net 11: JP3.6
- removed net 12: JP3.5
- removed net 6: JP3.9
- removed net N$31: R18.2, T8.B
- removed net N$32: R19.2, T9.B
- removed net N$33: R20.2, T10.B
- removed net N$34: R21.2, T11.B
- removed net N$35: R22.2, T12.B
- removed net N$36: R23.2, T13.B
- removed net N$37: IC2A.SER, IC3A.QH*
- removed net N$40: R15.1, T3.B
- removed net N$41: R14.1, T4.B
- removed net N$42: R13.2, T1.B
- removed net N$43: R12.2, T5.B
- removed net N$44: R11.2, T6.B
- new net N$46: IC5.P2, R26.1
- new net N$48: IC5.P3, R27.1
- new net N$49: IC5.P4, R28.1
- new net N$50: IC5.P5, R29.1
- new net N$51: IC5.P6, R30.1
- new net N$52: R24.2, T14.B
- new net N$53: R25.2, T15.B
- new net N$54: R26.2, T16.B
- new net N$55: R27.2, T17.B
- new net N$56: R28.2, T18.B
- new net N$57: R29.2, T19.B
- new net N$58: R30.2, T20.B
- new net N$59: IC4.P0, R38.2
- new net N$60: R36.1, T22.B
- new net N$61: R35.1, T23.B
- new net N$62: R34.1, T24.B
- new net N$63: R33.2, T21.B
- new net N$64: R32.2, T25.B
- new net N$65: R31.2, T26.B
- new net N$66: IC4.P1, R31.1
- new net N$67: IC4.P2, R32.1
- new net N$68: IC4.P3, R33.1
- new net N$69: IC4.P4, R34.2
- new net N$70: IC4.P5, R35.2
- new net N$71: IC4.P6, R36.2
- new net N$72: IC5.P7, R37.1
- new net N$73: R38.1, T27.B
- new net N$74: R37.2, T28.B
- net +3V3: now also IC4.VDD, IC5.VDD, T14.E, T15.E, T16.E, T17.E, T18.E, T19.E, T20.E, T28.E; no longer JP1.15
- net 13: no longer JP3.4
- net 2: no longer JP3.12
- net 3: no longer JP3.11
- net 5: no longer JP3.10
- net 9: no longer JP3.8
- net A0: no longer JP1.12
- net A1: no longer JP1.11
- net A2: no longer JP1.10
- net A3: no longer JP1.9
- net A4: now also IC4.SDA, IC5.SDA; no longer JP1.8
- net A5: now also IC4.SCL, IC5.SCL; no longer JP1.7
- net AREF: no longer JP1.14
- net DFU: no longer JP1.1
- net EN: no longer JP3.2
- net GND: now also IC4.VSS, IC5.VSS, T21.E, T22.E, T23.E, T24.E, T25.E, T26.E, T27.E; no longer JP1.13, T1.E, T2.E, T3.E, T4.E, T5.E, T6.E
- net MISO: no longer IC1.PB3(PDO/MISO), JP1.4
- net MOSI: no longer IC1.PB2(PDI/MOSI), JP1.5
- net N$10: now also J1.4, T17.C; no longer IC3A.QD, R13.1
- net N$13: now also J1.5, T18.C; no longer IC3A.QC, R12.1
- net N$14: now also J3.5, T22.C; no longer IC3A.QB, R11.1
- net N$19: now also J3.4, T23.C; no longer R16.1, T2.B
- net N$23: now also J3.3, T24.C; no longer IC2A.QB, R17.1
- net N$24: now also J3.2, T21.C; no longer IC2A.QC, R18.1
- net N$25: now also J3.1, T25.C; no longer IC2A.QD, R19.1
- net N$26: now also J2.5, T26.C; no longer IC2A.QE, R20.1
- net N$27: now also J2.4, T27.C; no longer IC2A.QF, R21.1
- net N$28: now also J2.2, T20.C; no longer IC2A.QG, R22.1
- net N$29: now also J2.3, T19.C; no longer IC2A.QH, R23.1
- net N$30: now also J2.1, T28.C; no longer R17.2, T7.B
- net N$38: now also IC5.P0, R24.1; no longer IC2A.SCK, IC3A.SCK
- net N$39: now also IC5.P1, R25.1; no longer IC2A.RCK, IC3A.RCK
- net N$7: now also J1.1, T14.C; no longer IC3A.QE, R14.2
- net N$8: now also J1.2, T15.C; no longer IC3A.QG, R16.2
- net N$9: now also J1.3, T16.C; no longer IC3A.QF, R15.2
- net RST: no longer JP1.16
- net SCK: no longer IC1.PB1(SCK), JP1.6
- net VBAT: no longer JP3.1
- net VBUS: no longer JP3.3
Other:
- moved on the sheet: C9, IC1, R4, R5, X3, Y1
